File: electronic/electronic.kicad_pcb (KiCad board)
At the start: 2 copper layers, 0 parts

Commit message: chore: ESP32 devkit changed of schematic
Parts:
- added J1: M_BAT01, Connector_JST:JST_XH_B2B-XH-A_1x02_P2.50mm_Vertical, F.Cu at (98.0, 33.5)
- added J10: BMP01, Connector_PinHeader_2.54mm:PinHeader_1x06_P2.54mm_Vertical, F.Cu at (144.8, 45.4)
- added J11: MPU6050_01, Connector_PinHeader_2.54mm:PinHeader_1x08_P2.54mm_Vertical, F.Cu at (140.2, 45.4)
- added J12: NEO_06_01, Connector_PinHeader_2.54mm:PinHeader_1x04_P2.54mm_Vertical, F.Cu at (155.0, 68.9)
- added J14: OLED, Connector_PinHeader_2.54mm:PinHeader_1x04_P2.54mm_Vertical, F.Cu at (141.0, 99.4)
- added J15: HCSR01, Connector_PinHeader_2.54mm:PinHeader_1x04_P2.54mm_Vertical, F.Cu at (130.6, 84.4)
- added J16: HCSR01, Connector_PinHeader_2.54mm:PinHeader_1x04_P2.54mm_Vertical, F.Cu at (135.2, 84.4)
- added J17: HCSR01, Connector_PinHeader_2.54mm:PinHeader_1x04_P2.54mm_Vertical, F.Cu at (139.8, 84.4)
- added J18: HCSR01, Connector_PinHeader_2.54mm:PinHeader_1x04_P2.54mm_Vertical, F.Cu at (144.5, 84.4)
- added J2: M_SIG01, Connector_JST:JST_XH_B2B-XH-A_1x02_P2.50mm_Vertical, F.Cu at (106.5, 33.5)
- added J3: M_SIG01, Connector_JST:JST_XH_B2B-XH-A_1x02_P2.50mm_Vertical, F.Cu at (122.4, 62.0)
- added J4: M_BAT01, Connector_JST:JST_XH_B2B-XH-A_1x02_P2.50mm_Vertical, F.Cu at (122.4, 69.8)
- added J5: M_SIG01, Connector_JST:JST_XH_B2B-XH-A_1x02_P2.50mm_Vertical, F.Cu at (122.4, 77.6)
- added J6: M_BAT01, Connector_JST:JST_XH_B2B-XH-A_1x02_P2.50mm_Vertical, F.Cu at (131.8, 46.4)
- added J7: M_SIG01, Connector_JST:JST_XH_B2B-XH-A_1x02_P2.50mm_Vertical, F.Cu at (131.8, 54.2)
- added J8: M_BAT01, Connector_JST:JST_XH_B2B-XH-A_1x02_P2.50mm_Vertical, F.Cu at (131.8, 62.0)
- added J9: DHT01, Connector_PinHeader_2.54mm:PinHeader_1x04_P2.54mm_Vertical, F.Cu at (121.2, 84.4)
- added R1: 10k, Resistor_THT:R_Axial_DIN0207_L6.3mm_D2.5mm_P10.16mm_Horizontal, F.Cu at (116.5, 94.2)
- added U10: DEVKIT_V1_ESP32-WROOM-32, custom:MODULE_DEVKIT_V1_ESP32-WROOM-32, F.Cu at (89.3, 67.6)
