Commit message: chore(fdrone): rename *_*.STL files to *.STL and add launcher for display the project in rviz2

File: ros-ws/src/fdrone/urdf/model.urdf (robot description, URDF)
Before this commit: robot URDF.SLDASM, 5 links, 4 joints
Links:
- link BASE_LINK: geometry collision mesh filename=file:///home/akey/Unix/projects/networks/ros-ws/src/fdrone/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; visual mesh filename=file:///home/akey/Unix/projects/networks/ros-ws/src/fdrone/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
- link LB_LINK: geometry collision mesh filename=file:///home/akey/Unix/projects/networks/ros-ws/src/fdrone/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; visual mesh filename=file:///home/akey/Unix/projects/networks/ros-ws/src/fdrone/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
- link LT_LINK: geometry collision mesh filename=file:///home/akey/Unix/projects/networks/ros-ws/src/fdrone/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; visual mesh filename=file:///home/akey/Unix/projects/networks/ros-ws/src/fdrone/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
- link RB_LINK: geometry collision mesh filename=file:///home/akey/Unix/projects/networks/ros-ws/src/fdrone/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; visual mesh filename=file:///home/akey/Unix/projects/networks/ros-ws/src/fdrone/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
- link RT_LINK: geometry collision mesh filename=file:///home/akey/Unix/projects/networks/ros-ws/src/fdrone/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; visual mesh filename=file:///home/akey/Unix/projects/networks/ros-ws/src/fdrone/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

Commit message: refactor (model.urdf): test gz-sim-multicopter-control-system plugin

File: ros-ws/src/fdrone/urdf/model.urdf (robot description, URDF)
Before this commit: robot URDF.SLDASM, 5 links, 4 joints
Links:
- removed link BASE_LINK
- removed link LB_LINK
- removed link LT_LINK
- removed link RB_LINK
- removed link RT_LINK
- added link base_link, mass 0.89737; collision mesh filename=file:///home/akey/Unix/projects/networks/ros-ws/src/fdrone/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; visual mesh filename=file:///home/akey/Unix/projects/networks/ros-ws/src/fdrone/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
- added link rotor_0, mass 0.005; collision mesh filename=file:///home/akey/Unix/projects/networks/ros-ws/src/fdrone/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; visual mesh filename=file:///home/akey/Unix/projects/networks/ros-ws/src/fdrone/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
- added link rotor_1, mass 0.005; collision mesh filename=file:///home/akey/Unix/projects/networks/ros-ws/src/fdrone/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; visual mesh filename=file:///home/akey/Unix/projects/networks/ros-ws/src/fdrone/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
- added link rotor_2, mass 0.005; collision mesh filename=file:///home/akey/Unix/projects/networks/ros-ws/src/fdrone/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; visual mesh filename=file:///home/akey/Unix/projects/networks/ros-ws/src/fdrone/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
- added link rotor_3, mass 0.005; collision mesh filename=file:///home/akey/Unix/projects/networks/ros-ws/src/fdrone/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; visual mesh filename=file:///home/akey/Unix/projects/networks/ros-ws/src/fdrone/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
- added link world
Joints:
- removed joint JX_00
- removed joint JX_01
- removed joint JX_02
- removed joint JX_03
- added joint rotor_0_joint: type revolute, parent base_link, child rotor_0, origin xyz=-0.15758 0.15891 0.11523 rpy=1.5708 0 0, axis 0 1 0, limit effort=0.03 velocity=870
- added joint rotor_1_joint: type revolute, parent base_link, child rotor_1, origin xyz=0.16023 0.1589 0.11523 rpy=1.5708 0 0, axis 0 1 0, limit effort=0.03 velocity=870
- added joint rotor_2_joint: type revolute, parent base_link, child rotor_2, origin xyz=0.16022 -0.15891 0.11523 rpy=1.5708 0 0, axis 0 1 0, limit effort=0.03 velocity=870
- added joint rotor_3_joint: type revolute, parent base_link, child rotor_3, origin xyz=-0.15759 -0.1589 0.11523 rpy=1.5708 0 0, axis 0 1 0, limit effort=0.03 velocity=870
- added joint world_to_base: type fixed, parent world, child base_link, origin xyz=0 0 0 rpy=0 0 0

Commit message: chore(ros-ws): test control of joints with gz-sim-joint-controller-system

File: ros-ws/src/fdrone/urdf/model.urdf (robot description, URDF)
Before this commit: robot URDF.SLDASM, 5 links, 4 joints
Links:
- added link world
- link LB_LINK: mass 0.89737 -> 0.01
- link LT_LINK: mass 0.89737 -> 0.01
- link RB_LINK: mass 0.89737 -> 0.01
- link RT_LINK: mass 0.89737 -> 0.01
Joints:
- added joint world_to_base: type fixed, parent world, child BASE_LINK, origin xyz=0 0 0 rpy=0 0 0
- joint JX_00: limit effort=0.03 velocity=870 -> effort=2.9 velocity=870
- joint JX_01: limit effort=0.03 velocity=870 -> effort=0.53 velocity=870
- joint JX_02: limit effort=0.03 velocity=870 -> effort=2.9 velocity=870
- joint JX_03: limit effort=0.03 velocity=870 -> effort=2.9 velocity=870

Commit message: fix(model.urdf): set test limit effort for joints

File: ros-ws/src/fdrone/urdf/model.urdf (robot description, URDF)
Before this commit: robot fdrone, 5 links, 4 joints
Joints:
- joint JX_01: limit effort=0.53 velocity=870 -> effort=2.9 velocity=870

Commit message: refactor(ros-ws): change names of topics, nodes and elements in the urdf

File: ros-ws/src/fdrone/urdf/model.urdf (robot description, URDF)
Before this commit: robot fdrone, 5 links, 4 joints
Links:
- removed link BASE_LINK
- removed link LB_LINK
- removed link LT_LINK
- removed link RB_LINK
- removed link RT_LINK
- added link base_link, mass 0.86; collision mesh filename=file:///home/akey/Unix/projects/networks/ros-ws/src/fdrone/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; visual mesh filename=file:///home/akey/Unix/projects/networks/ros-ws/src/fdrone/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
- added link rotor_0, mass 0.01; collision mesh filename=file:///home/akey/Unix/projects/networks/ros-ws/src/fdrone/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; visual mesh filename=file:///home/akey/Unix/projects/networks/ros-ws/src/fdrone/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
- added link rotor_1, mass 0.01; collision mesh filename=file:///home/akey/Unix/projects/networks/ros-ws/src/fdrone/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; visual mesh filename=file:///home/akey/Unix/projects/networks/ros-ws/src/fdrone/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
- added link rotor_2, mass 0.01; collision mesh filename=file:///home/akey/Unix/projects/networks/ros-ws/src/fdrone/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; visual mesh filename=file:///home/akey/Unix/projects/networks/ros-ws/src/fdrone/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
- added link rotor_3, mass 0.01; collision mesh filename=file:///home/akey/Unix/projects/networks/ros-ws/src/fdrone/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; visual mesh filename=file:///home/akey/Unix/projects/networks/ros-ws/src/fdrone/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
Joints:
- removed joint JX_00
- removed joint JX_01
- removed joint JX_02
- removed joint JX_03
- added joint rotor_0_joint: type continuous, parent base_link, child rotor_0, origin xyz=-0.15758 0.15891 0.11523 rpy=1.5708 0 0, axis 0 1 0, limit effort=3000 velocity=8700
- added joint rotor_1_joint: type continuous, parent base_link, child rotor_1, origin xyz=0.16023 0.1589 0.11523 rpy=1.5708 0 0, axis 0 1 0, limit effort=3000 velocity=8700
- added joint rotor_2_joint: type continuous, parent base_link, child rotor_2, origin xyz=0.16022 -0.15891 0.11523 rpy=1.5708 0 0, axis 0 1 0, limit effort=3000 velocity=8700
- added joint rotor_3_joint: type continuous, parent base_link, child rotor_3, origin xyz=-0.15759 -0.1589 0.11523 rpy=1.5708 0 0, axis 0 1 0, limit effort=3000 velocity=8700

Commit message: refactor(ros-ws): change the filename attrib in urdf to use relative directory based on the project

File: ros-ws/src/fdrone/urdf/model.urdf (robot description, URDF)
Before this commit: robot fdrone, 5 links, 4 joints
Links:
- link base_link: geometry collision mesh filename=file://$(find fdrone)/urdf/meshes/BASELINK.STL; visual mesh filename=file://$(find fdrone)/urdf/meshes/BASELINK.STL
- link rotor_0: geometry collision mesh filename=file://$(find fdrone)/urdf/meshes/RTLINK.STL; visual mesh filename=file://$(find fdrone)/urdf/meshes/RTLINK.STL
- link rotor_1: geometry collision mesh filename=file://$(find fdrone)/urdf/meshes/RBLINK.STL; visual mesh filename=file://$(find fdrone)/urdf/meshes/RBLINK.STL
- link rotor_2: geometry collision mesh filename=file://$(find fdrone)/urdf/meshes/LBLINK.STL; visual mesh filename=file://$(find fdrone)/urdf/meshes/LBLINK.STL
- link rotor_3: geometry collision mesh filename=file://$(find fdrone)/urdf/meshes/LTLINK.STL; visual mesh filename=file://$(find fdrone)/urdf/meshes/LTLINK.STL

Commit message: chore(ros-ws): update UAV base

File: ros-ws/src/fdrone/urdf/model.urdf (robot description, URDF)
Before this commit: robot fdrone, 5 links, 4 joints
Links:
- link base_link: mass 0.86 -> 1.20
Joints:
- joint rotor_0_joint: limit effort=3000 velocity=8700 -> effort=1e6 velocity=8700; origin xyz=-0.15758 0.15891 0.11523 rpy=1.5708 0 0 -> xyz=-0.1589 0.1589 0.13673 rpy=1.5708 0 0
- joint rotor_1_joint: limit effort=3000 velocity=8700 -> effort=1e6 velocity=8700; origin xyz=0.16023 0.1589 0.11523 rpy=1.5708 0 0 -> xyz=0.1589 0.1589 0.13673 rpy=1.5708 0 0
- joint rotor_2_joint: limit effort=3000 velocity=8700 -> effort=1e6 velocity=8700; origin xyz=0.16022 -0.15891 0.11523 rpy=1.5708 0 0 -> xyz=0.1589 -0.1589 0.13673 rpy=1.5708 0 0
- joint rotor_3_joint: limit effort=3000 velocity=8700 -> effort=1e6 velocity=8700; origin xyz=-0.15759 -0.1589 0.11523 rpy=1.5708 0 0 -> xyz=-0.1589 -0.1589 0.13673 rpy=1.5708 0 0
